File: Hardware/MiP_Mini-Pack.brd (EAGLE design)
At the start: 41.4 x 63.8 mm, 41 parts, among them Q1 8MHz, U1 ATMEGA328, U3 TS3USB221A

Commit message: corrected labels, ready for review
Parts:
- added C10: 0.1uF, SparkFun:0603-CAP
- added C13, C19: 10uF, SparkFun:EIA3216
- added U2: MIC5205, SparkFun:SOT23-5
- moved LOGO1 46.0 mm to (15.4, 54.9)
- moved LOGO2 13.3 mm to (17.8, 44.2)
- moved F1 12.5 mm to (3.17, 24.1), turned to 90 degrees
- moved D4 1.78 mm to (29.6, 15.5)
Connections:
- net GND: now also C10.2, C13.C, C19.C, U2.2
- net VCC: now also C10.1, C13.A, U2.5
- net VIN: now also C19.A, U2.1, U2.3
Routing:
- net N$17: track 16.1 -> 2.52 mm
- net VCC: track 126.9 -> 134.8 mm, vias 3 -> 4
- net VIN: track 90.5 -> 93.0 mm, vias 0 -> 2
- net N$8: track 1.70 -> 3.48 mm
- net SELECT: track 16.4 -> 15.7 mm
- added copper zone on layer 1, net VIN
